File: ws2812_2020_pyramid.sch (KiCad schematic (older format))
At the start: 50 parts

Commit message: Finish design
Parts:
- D1, D10, D11, D12, D13, D14, D15, D16, D17, D18, D19, D2, D20, D21, D22, D23, D24, D25, D26, D27, D28, D29, D3, D30, D31, D32, D33, D34, D35, D36, D4, D5, D6, D7, D8, D9: symbol LED:WS2812B -> WM_lib:WS2812_2020-LED
Connections:
- net +5V: now also D1.4 (VDD), D10.4 (VDD), D11.4 (VDD), D12.4 (VDD), D13.4 (VDD), D14.4 (VDD), D15.4 (VDD), D16.4 (VDD), D17.4 (VDD), D18.4 (VDD), D19.4 (VDD), D2.4 (VDD), D20.4 (VDD), D21.4 (VDD), D22.4 (VDD), D23.4 (VDD), D24.4 (VDD), D25.4 (VDD), D26.4 (VDD), D27.4 (VDD), D28.4 (VDD), D29.4 (VDD), D3.4 (VDD), D30.4 (VDD), D31.4 (VDD), D32.4 (VDD), D33.4 (VDD), D34.4 (VDD), D35.4 (VDD), D36.4 (VDD), D4.4 (VDD), D5.4 (VDD), D6.4 (VDD), D7.4 (VDD), D8.4 (VDD), D9.4 (VDD); no longer D1.1 (VDD), D10.1 (VDD), D11.1 (VDD), D12.1 (VDD), D13.1 (VDD), D14.1 (VDD), D15.1 (VDD), D16.1 (VDD), D17.1 (VDD), D18.1 (VDD), D19.1 (VDD), D2.1 (VDD), D20.1 (VDD), D21.1 (VDD), D22.1 (VDD), D23.1 (VDD), D24.1 (VDD), D25.1 (VDD), D26.1 (VDD), D27.1 (VDD), D28.1 (VDD), D29.1 (VDD), D3.1 (VDD), D30.1 (VDD), D31.1 (VDD), D32.1 (VDD), D33.1 (VDD), D34.1 (VDD), D35.1 (VDD), D36.1 (VDD), D4.1 (VDD), D5.1 (VDD), D6.1 (VDD), D7.1 (VDD), D8.1 (VDD), D9.1 (VDD)
- net DIN: now also D1.3 (DIN); no longer D1.4 (DIN)
- net DOUT: now also D36.1 (DOUT); no longer D36.2 (DOUT)
- net GND: now also D1.2 (GND), D10.2 (GND), D11.2 (GND), D12.2 (GND), D13.2 (GND), D14.2 (GND), D15.2 (GND), D16.2 (GND), D17.2 (GND), D18.2 (GND), D19.2 (GND), D2.2 (GND), D20.2 (GND), D21.2 (GND), D22.2 (GND), D23.2 (GND), D24.2 (GND), D25.2 (GND), D26.2 (GND), D27.2 (GND), D28.2 (GND), D29.2 (GND), D3.2 (GND), D30.2 (GND), D31.2 (GND), D32.2 (GND), D33.2 (GND), D34.2 (GND), D35.2 (GND), D36.2 (GND), D4.2 (GND), D5.2 (GND), D6.2 (GND), D7.2 (GND), D8.2 (GND), D9.2 (GND); no longer D1.3 (VSS), D10.3 (VSS), D11.3 (VSS), D12.3 (VSS), D13.3 (VSS), D14.3 (VSS), D15.3 (VSS), D16.3 (VSS), D17.3 (VSS), D18.3 (VSS), D19.3 (VSS), D2.3 (VSS), D20.3 (VSS), D21.3 (VSS), D22.3 (VSS), D23.3 (VSS), D24.3 (VSS), D25.3 (VSS), D26.3 (VSS), D27.3 (VSS), D28.3 (VSS), D29.3 (VSS), D3.3 (VSS), D30.3 (VSS), D31.3 (VSS), D32.3 (VSS), D33.3 (VSS), D34.3 (VSS), D35.3 (VSS), D36.3 (VSS), D4.3 (VSS), D5.3 (VSS), D6.3 (VSS), D7.3 (VSS), D8.3 (VSS), D9.3 (VSS)
- new net: D1.1 (DOUT), D2.3 (DIN)
- new net: D2.1 (DOUT), D3.3 (DIN)
- new net: D3.1 (DOUT), D4.3 (DIN)
- new net: D4.1 (DOUT), D5.3 (DIN)
- new net: D5.1 (DOUT), D6.3 (DIN)
- new net: D6.1 (DOUT), D7.3 (DIN)
- new net: D7.1 (DOUT), D8.3 (DIN)
- new net: D8.1 (DOUT), D9.3 (DIN)
- new net: D10.3 (DIN), D9.1 (DOUT)
- new net: D10.1 (DOUT), D11.3 (DIN)
- new net: D11.1 (DOUT), D12.3 (DIN)
- new net: D12.1 (DOUT), D13.3 (DIN)
- new net: D13.1 (DOUT), D14.3 (DIN)
- new net: D14.1 (DOUT), D15.3 (DIN)
- new net: D15.1 (DOUT), D16.3 (DIN)
- new net: D16.1 (DOUT), D17.3 (DIN)
- new net: D17.1 (DOUT), D18.3 (DIN)
- new net: D18.1 (DOUT), D19.3 (DIN)
- new net: D19.1 (DOUT), D20.3 (DIN)
- new net: D20.1 (DOUT), D21.3 (DIN)
- new net: D21.1 (DOUT), D22.3 (DIN)
- new net: D25.1 (DOUT), D26.3 (DIN)
- new net: D24.1 (DOUT), D25.3 (DIN)
- new net: D26.1 (DOUT), D27.3 (DIN)
- new net: D27.1 (DOUT), D28.3 (DIN)
- new net: D28.1 (DOUT), D29.3 (DIN)
- new net: D29.1 (DOUT), D30.3 (DIN)
- new net: D30.1 (DOUT), D31.3 (DIN)
- new net: D31.1 (DOUT), D32.3 (DIN)
- new net: D22.1 (DOUT), D23.3 (DIN)
- new net: D23.1 (DOUT), D24.3 (DIN)
- new net: D32.1 (DOUT), D33.3 (DIN)
- new net: D33.1 (DOUT), D34.3 (DIN)
- new net: D34.1 (DOUT), D35.3 (DIN)
- new net: D35.1 (DOUT), D36.3 (DIN)
Changed lines of the file:
@@
 $EndComp
 $Comp
-L LED:WS2812B D2
+L WM_lib:WS2812_2020-LED D2
 U 1 1 5F9C4526
 P 4600 2450
@@
 $EndComp
 $Comp
-L LED:WS2812B D3
+L WM_lib:WS2812_2020-LED D3
 U 1 1 5F9C4913
 P 5350 2450
@@
 $EndComp
 $Comp
-L LED:WS2812B D4
+L WM_lib:WS2812_2020-LED D4
 U 1 1 5F9C4EA8
 P 6100 2450
@@
 $EndComp
 $Comp
-L LED:WS2812B D5
+L WM_lib:WS2812_2020-LED D5
 U 1 1 5F9C8ACD
 P 3850 3400
@@
 $EndComp
 $Comp
-L LED:WS2812B D6
+L WM_lib:WS2812_2020-LED D6
 U 1 1 5F9C8AD3
 P 4600 3400
@@
 $EndComp
 $Comp
-L LED:WS2812B D7
+L WM_lib:WS2812_2020-LED D7
 U 1 1 5F9C8AD9
 P 5350 3400
@@
 $EndComp
 $Comp
-L LED:WS2812B D8
+L WM_lib:WS2812_2020-LED D8
 U 1 1 5F9CA604
 P 6100 3400
@@
 $EndComp
 $Comp
-L LED:WS2812B D9
+L WM_lib:WS2812_2020-LED D9
 U 1 1 5F9CA60A
 P 6850 3400
@@
 $EndComp
 $Comp
-L LED:WS2812B D10
+L WM_lib:WS2812_2020-LED D10
 U 1 1 5F9CED20
 P 3100 4100
@@
 $EndComp
 $Comp
-L LED:WS2812B D11
+L WM_lib:WS2812_2020-LED D11
 U 1 1 5F9CED26
 P 3850 4100
@@
 $EndComp
 $Comp
-L LED:WS2812B D12
+L WM_lib:WS2812_2020-LED D12
 U 1 1 5F9CED2C
 P 4600 4100
@@
 $EndComp
 $Comp
-L LED:WS2812B D13
+L WM_lib:WS2812_2020-LED D13
 U 1 1 5F9CED32
 P 5350 4100
@@
 $EndComp
 $Comp
-L LED:WS2812B D14
+L WM_lib:WS2812_2020-LED D14
 U 1 1 5F9CED38
 P 6100 4100
@@
 $EndComp
 $Comp
-L LED:WS2812B D15
+L WM_lib:WS2812_2020-LED D15
 U 1 1 5F9CFB04
 P 6850 4100
@@
 $EndComp
 $Comp
-L LED:WS2812B D16
+L WM_lib:WS2812_2020-LED D16
 U 1 1 5F9CFB0A
 P 7600 4100
@@
 	9000 3800 9000 3900
 $Comp
-L LED:WS2812B D17
+L WM_lib:WS2812_2020-LED D17
 U 1 1 5FA164ED
 P 2350 4950
@@
 $EndComp
 $Comp
-L LED:WS2812B D18
+L WM_lib:WS2812_2020-LED D18
 U 1 1 5FA164F3
 P 3100 4950
@@
 $EndComp
 $Comp
-L LED:WS2812B D19
+L WM_lib:WS2812_2020-LED D19
 U 1 1 5FA164F9
 P 3850 4950
@@
 $EndComp
 $Comp
-L LED:WS2812B D20
+L WM_lib:WS2812_2020-LED D20
 U 1 1 5FA164FF
 P 4600 4950
@@
 $EndComp
 $Comp
-L LED:WS2812B D21
+L WM_lib:WS2812_2020-LED D21
 U 1 1 5FA16505
 P 5350 4950
@@
 $EndComp
 $Comp
-L LED:WS2812B D25
+L WM_lib:WS2812_2020-LED D25
 U 1 1 5FA1650B
 P 8350 4950
@@
 $EndComp
 $Comp
-L LED:WS2812B D26
+L WM_lib:WS2812_2020-LED D26
 U 1 1 5FA16511
 P 1600 5650
@@
 $EndComp
 $Comp
-L LED:WS2812B D27
+L WM_lib:WS2812_2020-LED D27
 U 1 1 5FA16517
 P 2350 5650
@@
 $EndComp
 $Comp
-L LED:WS2812B D28
+L WM_lib:WS2812_2020-LED D28
 U 1 1 5FA1651D
 P 3100 5650
@@
 $EndComp
 $Comp
-L LED:WS2812B D29
+L WM_lib:WS2812_2020-LED D29
 U 1 1 5FA16523
 P 3850 5650
@@
 $EndComp
 $Comp
-L LED:WS2812B D30
+L WM_lib:WS2812_2020-LED D30
 U 1 1 5FA16529
 P 4600 5650
@@
 $EndComp
 $Comp
-L LED:WS2812B D31
+L WM_lib:WS2812_2020-LED D31
 U 1 1 5FA1652F
 P 5350 5650
@@
 $EndComp
 $Comp
-L LED:WS2812B D22
+L WM_lib:WS2812_2020-LED D22
 U 1 1 5FA18B3B
 P 6100 4950
@@
 $EndComp
 $Comp
-L LED:WS2812B D23
+L WM_lib:WS2812_2020-LED D23
 U 1 1 5FA18B41
 P 6850 4950
@@
 $EndComp
 $Comp
-L LED:WS2812B D24
+L WM_lib:WS2812_2020-LED D24
 U 1 1 5FA18B47
 P 7600 4950
@@
 $EndComp
 $Comp
-L LED:WS2812B D32
+L WM_lib:WS2812_2020-LED D32
 U 1 1 5FA1A70C
 P 6100 5650
@@
 +5V
 $Comp
-L LED:WS2812B D1
+L WM_lib:WS2812_2020-LED D1
 U 1 1 5F9C23F8
 P 5350 1700
@@
 	7600 5950 6850 5950
 $Comp
-L LED:WS2812B D34
+L WM_lib:WS2812_2020-LED D34
 U 1 1 5FA1A718
 P 7600 5650
@@
 $EndComp
 $Comp
-L LED:WS2812B D33
+L WM_lib:WS2812_2020-LED D33
 U 1 1 5FA1A712
 P 6850 5650
@@
 	1200 5300 8850 5300
 $Comp
-L LED:WS2812B D36
+L WM_lib:WS2812_2020-LED D36
 U 1 1 5FBE0140
 P 9100 5650
@@
 $EndComp
 $Comp
-L LED:WS2812B D35
+L WM_lib:WS2812_2020-LED D35
 U 1 1 5FBE0146
 P 8350 5650
